Commit message: added remote control and ackermann emulator. Closes: #7.

File: robot_sim/urdf/tas_car.urdf.xacro (robot description, xacro)
@@ -21,5 +21,5 @@
     </collision>
     <inertial>
-      <mass value="2.0"/>
+      <mass value="80.0"/>
       <inertia ixx="0.37267" ixy="0.535" ixz="0.27612" iyy="0.60173" iyz="0.37267" izz="0.5256" />
     </inertial>
@@ -32,6 +32,6 @@
   </joint>
   <!-- create the wheels -->
-  <xacro:r_wheel name="r_f_wheel" parent="base" joint_xyz="0.172 0.19189 -0.009168" joint_rpy="${PI/2} 0 0"/>
-  <xacro:l_wheel name="l_f_wheel" parent="base" joint_xyz="0.172 -0.19189 -0.009168" joint_rpy="${PI/2} 0 0"/>
+  <xacro:r_front_wheel name="r_f_wheel" parent="base" joint_xyz="0.172 0.19189 -0.009168" joint_rpy="${PI/2} 0 0"/>
+  <xacro:l_front_wheel name="l_f_wheel" parent="base" joint_xyz="0.172 -0.19189 -0.009168" joint_rpy="${PI/2} 0 0"/>
   <xacro:r_wheel name="r_b_wheel" parent="base" joint_xyz="-0.18673 0.19189 -0.009168" joint_rpy="${PI/2} 0 0"/>
   <xacro:l_wheel name="l_b_wheel" parent="base" joint_xyz="-0.18673 -0.19189 -0.009168" joint_rpy="${PI/2} 0 0"/>
@@ -58,4 +58,6 @@
   <xacro:transmission_block joint_name="base_r_b_wheel_joint" interface_type="EffortJointInterface"/>
   <xacro:transmission_block joint_name="base_l_b_wheel_joint" interface_type="EffortJointInterface"/>
+  <xacro:transmission_block joint_name="base_r_f_wheel_dummy_joint" interface_type="EffortJointInterface"/>
+  <xacro:transmission_block joint_name="base_l_f_wheel_dummy_joint" interface_type="EffortJointInterface"/>
   <xacro:ros_control_plugin ns="/tas_car"/>
   <!-- Gazebo ground truth position publisher -->

File: robot_sim/urdf/tas_car_macros.xacro (robot description, xacro)
@@ -24,4 +24,5 @@
     </link>
     <joint name="${parent}_${name}_joint" type="${act_type}">
+      <limit effort="1000000" velocity="100"/>
       <axis xyz="0 0 1" rpy="0 0 0"/>
       <origin xyz="${joint_xyz}" rpy="${joint_rpy}"/>
@@ -30,4 +31,57 @@
     </joint>
   </xacro:macro>
+  <!-- Right front wheel macro. Emulates ackermann drive. -->
+  <xacro:macro name="r_front_wheel" params="name xyz:='0 0 0' rpy:='0 0 0' mass:='0.0482' parent joint_xyz joint_rpy act_type:='continuous'">
+    <link name="${name}_dummy_link">
+      <visual>
+	<origin xyz="0 0 0" rpy="0 0 0"/>
+        <geometry>
+	  <box size="0.01 0.01 0.01"/>
+	</geometry>
+       </visual>
+      <collision>
+        <geometry>
+	  <box size="0.01 0.01 0.01"/>
+        </geometry>
+      </collision>
+      <inertial>
+	<mass value="0.1"/>
+	<origin xyz="0 0 0" />
+	<inertia ixx="3.745e-7" ixy="6.657e-7" ixz="3.28e-7" iyy="3.28e-7" iyz="3.745e-7" izz="6.657e-7"/>
+      </inertial>
+    </link>
+    <joint name="${parent}_${name}_dummy_joint" type="${act_type}">
+      <limit effort="1000000" velocity="100"/>
+      <axis xyz="0 0 1" rpy="0 0 0"/>
+      <origin xyz="${joint_xyz}" rpy="0 0 0"/>
+      <parent link="${parent}"/>
+      <child link="${name}_dummy_link"/>
+    </joint>
+    <link name="${name}">
+      <visual>
+	<origin xyz="${xyz}" rpy="${rpy}"/>
+        <geometry>
+	  <mesh filename="${wheel_r_mesh}"/>
+	</geometry>
+       </visual>
+      <collision>
+        <geometry>
+	  <mesh filename="${wheel_r_mesh_col}"/>
+        </geometry>
+      </collision>
+      <inertial>
+	<mass value="${mass}" />
+	<origin xyz="${xyz}" />
+	<inertia ixx="3.745e-7" ixy="6.657e-7" ixz="3.28e-7" iyy="3.28e-7" iyz="3.745e-7" izz="6.657e-7"/>
+      </inertial>
+    </link>
+    <joint name="${name}_dummy_${name}_joint" type="${act_type}">
+      <limit effort="1000000" velocity="100"/>
+      <axis xyz="0 0 1" rpy="0 0 0"/>
+      <origin xyz="0 0 0" rpy="${joint_rpy}"/>
+      <parent link="${name}_dummy_link"/>
+      <child link="${name}"/>
+    </joint>
+  </xacro:macro>
   <!-- Left wheel macro -->
   <xacro:macro name="l_wheel" params="name xyz:='0 0 0' rpy:='0 0 0' mass:='0.0482' parent joint_xyz joint_rpy act_type:='continuous'">
@@ -51,4 +105,5 @@
     </link>
     <joint name="${parent}_${name}_joint" type="${act_type}">
+      <limit effort="1000000" velocity="100"/>
       <axis xyz="0 0 1" rpy="0 0 0"/>
       <origin xyz="${joint_xyz}" rpy="${joint_rpy}"/>
@@ -57,4 +112,57 @@
     </joint>
   </xacro:macro>
+  <!-- Left front wheel macro. Emulates ackermann drive. -->
+  <xacro:macro name="l_front_wheel" params="name xyz:='0 0 0' rpy:='0 0 0' mass:='0.0482' parent joint_xyz joint_rpy act_type:='continuous'">
+    <link name="${name}_dummy_link">
+      <visual>
+	<origin xyz="0 0 0" rpy="0 0 0"/>
+        <geometry>
+	  <box size="0.01 0.01 0.01"/>
+	</geometry>
+       </visual>
+      <collision>
+        <geometry>
+	  <box size="0.01 0.01 0.01"/>
+        </geometry>
+      </collision>
+      <inertial>
+	<mass value="0.1"/>
+	<origin xyz="0 0 0" />
+	<inertia ixx="3.745e-7" ixy="6.657e-7" ixz="3.28e-7" iyy="3.28e-7" iyz="3.745e-7" izz="6.657e-7"/>
+      </inertial>
+    </link>
+    <joint name="${parent}_${name}_dummy_joint" type="${act_type}">
+      <limit effort="1000000" velocity="100"/>
+      <axis xyz="0 0 1" rpy="0 0 0"/>
+      <origin xyz="${joint_xyz}" rpy="0 0 0"/>
+      <parent link="${parent}"/>
+      <child link="${name}_dummy_link"/>
+    </joint>
+    <link name="${name}">
+      <visual>
+	<origin xyz="${xyz}" rpy="${rpy}"/>
+        <geometry>
+	  <mesh filename="${wheel_l_mesh}"/>
+	</geometry>
+       </visual>
+      <collision>
+        <geometry>
+	  <mesh filename="${wheel_l_mesh_col}"/>
+        </geometry>
+      </collision>
+      <inertial>
+	<mass value="${mass}" />
+	<origin xyz="${xyz}" />
+	<inertia ixx="3.745e-7" ixy="6.657e-7" ixz="3.28e-7" iyy="3.28e-7" iyz="3.745e-7" izz="6.657e-7"/>
+      </inertial>
+    </link>
+    <joint name="${name}_dummy_${name}_joint" type="${act_type}">
+      <limit effort="1000000" velocity="100"/>
+      <axis xyz="0 0 1" rpy="0 0 0"/>
+      <origin xyz="0 0 0" rpy="${joint_rpy}"/>
+      <parent link="${name}_dummy_link"/>
+      <child link="${name}"/>
+    </joint>
+  </xacro:macro>
   <!-- Hokuyo laser scanner macro -->
   <xacro:macro name="sensor_hokuyo" params="parent name:='hokuyo1' xyz:='0.08 0 0.430' rpy:='0 0 0'">
@@ -74,5 +182,5 @@
       </collision>
       <inertial>
-	<mass value="0.001"/>
+	<mass value="0.01"/>
 	<origin xyz="0 0 0"/>
 	<inertia ixx="0.0001" ixy="0.0" ixz="0.0" iyy="0.0001" iyz="0.0" izz="0.0001"/>
@@ -115,4 +223,5 @@
     </gazebo>
     <joint name="${name}_joint" type="fixed">
+      <limit effort="1000000" velocity="100"/>
       <origin xyz="${xyz}" rpy="${rpy}"/>
       <axis xyz="0 0 1" rpy="0 0 0"/>
