Commit message: fully functional sim. Closes: #11. Still not sure about #14

File: robot_sim/urdf/tas_car_macros.xacro (robot description, xacro)
@@ -277,5 +277,5 @@
     <joint name="base_cam_link_joint" type="fixed">
       <axis xyz="0 0 1" rpy="0 0 0"/>
-      <origin xyz="0.2 0 0.1" rpy="0 0 0"/>
+      <origin xyz="0.3 0 0.1" rpy="0 0 0"/>
       <parent link="base"/>
       <child link="cam_link"/>
